File: Placas/Placa Definitiva/v0.1/v0.1.kicad_pcb (KiCad board)
At the start: 2 copper layers, 4 parts, among them U1 ADC1175CIMTC/NOPB, U2 MCP6291T-E_OT

Commit message: skere
Parts:
- removed U2: MCP6291T-E_OT, MCP6291T-E_OT:SOT95P280X145-5N
- added C1: 10uF, Capacitor_Tantalum_SMD:CP_EIA-3528-15_AVX-H_Pad1.50x2.35mm_HandSolder, F.Cu at (82.6, 131.9)
- added C11: 100nF, Capacitor_SMD:C_0805_2012Metric_Pad1.18x1.45mm_HandSolder, F.Cu at (124.5, 104.4)
- added C12: 10uF, Capacitor_Tantalum_SMD:CP_EIA-3528-15_AVX-H_Pad1.50x2.35mm_HandSolder, F.Cu at (124.8, 99.6)
- added C13: 10uF, Capacitor_Tantalum_SMD:CP_EIA-3528-15_AVX-H_Pad1.50x2.35mm_HandSolder, F.Cu at (68.9, 103.0)
- added C14: 100nF, Capacitor_SMD:C_0805_2012Metric_Pad1.18x1.45mm_HandSolder, F.Cu at (64.8, 103.6)
- added C15: 10nF, Capacitor_SMD:C_0805_2012Metric_Pad1.18x1.45mm_HandSolder, F.Cu at (114.4, 71.4)
- added C2: 100nF, Capacitor_SMD:C_0805_2012Metric_Pad1.18x1.45mm_HandSolder, F.Cu at (78.3, 132.5)
- added C3: 10uF, Capacitor_Tantalum_SMD:CP_EIA-3528-15_AVX-H_Pad1.50x2.35mm_HandSolder, F.Cu at (59.1, 129.7)
- added C4: 100nF, Capacitor_SMD:C_0805_2012Metric_Pad1.18x1.45mm_HandSolder, F.Cu at (54.4, 130.2)
- added C5: 100uF, Capacitor_SMD:CP_Elec_6.3x7.7, F.Cu at (119.5, 64.4)
- added C6: 100nF, Capacitor_SMD:C_0805_2012Metric_Pad1.18x1.45mm_HandSolder, F.Cu at (126.0, 62.7)
- added C7: 10uF, Capacitor_Tantalum_SMD:CP_EIA-3528-15_AVX-H_Pad1.50x2.35mm_HandSolder, F.Cu at (121.1, 83.3)
- added C8: 100nF, Capacitor_SMD:C_0805_2012Metric_Pad1.18x1.45mm_HandSolder, F.Cu at (120.4, 87.2)
- added D1: BAT54C, Package_TO_SOT_SMD:SOT-23, F.Cu at (65.9, 60.9)
- added D2: BAT54C, Package_TO_SOT_SMD:SOT-23, F.Cu at (65.9, 66.3)
- added D3: BAT54C, Package_TO_SOT_SMD:SOT-23, F.Cu at (65.9, 71.6)
- added D4: BAT54C, Package_TO_SOT_SMD:SOT-23, F.Cu at (65.9, 77.0)
- added D5: BAT54C, Package_TO_SOT_SMD:SOT-23, F.Cu at (65.9, 82.3)
- added D6: BAT54C, Package_TO_SOT_SMD:SOT-23, F.Cu at (65.9, 87.7)
- added D7: BAT54C, Package_TO_SOT_SMD:SOT-23, F.Cu at (65.9, 93.0)
- added D8: BAT54C, Package_TO_SOT_SMD:SOT-23, F.Cu at (65.9, 98.4)
- added F1: Fuse, Fuse:Fuse_1206_3216Metric_Pad1.42x1.75mm_HandSolder, F.Cu at (112.0, 61.7)
- added IC1: SN74LVTH245ADWR, SN74LVTH245A-DWR:SOIC127P1030X265-20N, F.Cu at (76.3, 114.9)
- added IC2: ADA4891-1ARJZ-RL, ADA4891-1ARJZ-RL:SOT95P280X145-5N, F.Cu at (58.9, 103.5)
- added J1: Conn_01x09_Pin, Connector_PinHeader_2.54mm:PinHeader_1x09_P2.54mm_Vertical, F.Cu at (51.9, 60.8)
- added J2: Screw_Terminal_01x02, TerminalBlock:TerminalBlock_bornier-2_P5.08mm, F.Cu at (113.2, 85.4)
- added L1: 330uH, Inductor_SMD:L_Sunlord_SWRB1205S, F.Cu at (91.5, 131.0)
- added L2: 330uH, Inductor_SMD:L_Sunlord_SWRB1205S, F.Cu at (69.0, 131.3)
- added Q1: BC807, Package_TO_SOT_SMD:SOT-23, F.Cu at (59.7, 60.9)
- added Q2: BC807, Package_TO_SOT_SMD:SOT-23, F.Cu at (59.7, 66.3)
- added Q3: BC807, Package_TO_SOT_SMD:SOT-23, F.Cu at (59.7, 71.6)
- added Q4: BC807, Package_TO_SOT_SMD:SOT-23, F.Cu at (59.7, 77.0)
- added Q5: BC807, Package_TO_SOT_SMD:SOT-23, F.Cu at (59.7, 82.3)
- added Q6: BC807, Package_TO_SOT_SMD:SOT-23, F.Cu at (59.7, 87.7)
- added Q7: BC807, Package_TO_SOT_SMD:SOT-23, F.Cu at (59.7, 93.0)
- added Q8: BC807, Package_TO_SOT_SMD:SOT-23, F.Cu at (59.8, 98.4)
- added R3: 150k, Resistor_SMD:R_1206_3216Metric_Pad1.30x1.75mm_HandSolder, F.Cu at (53.3, 121.6)
- added R4: 150k, Resistor_SMD:R_1206_3216Metric_Pad1.30x1.75mm_HandSolder, F.Cu at (58.5, 121.6)
- added R5: 150k, Resistor_SMD:R_1206_3216Metric_Pad1.30x1.75mm_HandSolder, F.Cu at (114.7, 74.8)
- added U3: Raspberry Pi Pico, RaspberryPiPico:MODULE_SC0915, F.Cu at (95.9, 85.8)
- added U4: LM358, Package_SO:SOIC-8_3.9x4.9mm_P1.27mm, F.Cu at (55.0, 114.6)
- added U5: AMS1117-3.3, Package_TO_SOT_SMD:SOT-223-3_TabPin2, F.Cu at (122.8, 75.3)
- added U6: MAX9108ESD_, MAX9108ESD_:SOIC127P600X175-14N, F.Cu at (74.0, 63.5)
- added U7: MAX9108ESD_, MAX9108ESD_:SOIC127P600X175-14N, F.Cu at (73.9, 81.8)
- added U8: MCP4821, Package_SO:SOIC-8_3.9x4.9mm_P1.27mm, F.Cu at (115.2, 102.3)
- R1, R2: value R -> 150; footprint Resistor_THT:R_Axial_DIN0411_L9.9mm_D3.6mm_P12.70mm_Horizontal -> Resistor_SMD:R_1206_3216Metric_Pad1.30x1.75mm_HandSolder
- moved R1 109.8 mm to (60.0, 108.2)
- moved U1 106.4 mm to (64.5, 114.8), turned to 180 degrees
- moved R2 103.0 mm to (65.6, 108.2)
Connections:
- R1 pad 1: unconnected-(R1-Pad1) -> Net-(IC2--IN)
- R1 pad 2: unconnected-(R1-Pad2) -> /ADC_MCU
- R2 pad 1: unconnected-(R2-Pad1) -> /ADC_MCU
- R2 pad 2: unconnected-(R2-Pad2) -> GND
- U1 pad 1: unconnected-(U1-~OE-Pad1) -> GND
- U1 pad 10: unconnected-(U1-D7-Pad10) -> Net-(IC1-A8)
- U1 pad 11: unconnected-(U1-DVDD-Pad11) -> +5VD
- U1 pad 12: unconnected-(U1-CLK-Pad12) -> /ADC_CLK
- U1 pad 13: unconnected-(U1-DVDD-Pad13) -> +5VD
- U1 pad 14: unconnected-(U1-AVDD-Pad14) -> +5VA
- U1 pad 15: unconnected-(U1-AVDD-Pad15) -> +5VA
- U1 pad 17: unconnected-(U1-VRT-Pad17) -> /ADC_TOP_REF
- U1 pad 18: unconnected-(U1-AVDD-Pad18) -> +5VA
- U1 pad 19: unconnected-(U1-VIN-Pad19) -> /ADC_MCU
- U1 pad 2: unconnected-(U1-DVSS-Pad2) -> GND
- U1 pad 20: unconnected-(U1-AVSS-Pad20) -> GND
- U1 pad 21: unconnected-(U1-AVSS-Pad21) -> GND
- U1 pad 23: unconnected-(U1-VRB-Pad23) -> GND
- U1 pad 24: unconnected-(U1-DVSS-Pad24) -> GND
- U1 pad 3: unconnected-(U1-D0-Pad3) -> Net-(IC1-A1)
- U1 pad 4: unconnected-(U1-D1-Pad4) -> Net-(IC1-A2)
- U1 pad 5: unconnected-(U1-D2-Pad5) -> Net-(IC1-A3)
- U1 pad 6: unconnected-(U1-D3-Pad6) -> Net-(IC1-A4)
- U1 pad 7: unconnected-(U1-D4-Pad7) -> Net-(IC1-A5)
- U1 pad 8: unconnected-(U1-D5-Pad8) -> Net-(IC1-A6)
- U1 pad 9: unconnected-(U1-D6-Pad9) -> Net-(IC1-A7)
Routing:
- net +5V: track 0.00 -> 247.3 mm, vias 0 -> 14
- net +3.3V: track 0.00 -> 131.8 mm, vias 0 -> 3
- net /DAC_OUT: track 0.00 -> 126.4 mm, vias 0 -> 2
- net /ADC_MCU: track 0.00 -> 79.8 mm, vias 0 -> 2
- net Net-(IC2-+IN): track 0.00 -> 71.8 mm, vias 0 -> 2
- net /ADC_CLK: track 0.00 -> 61.5 mm, vias 0 -> 2
- net +5VD: track 0.00 -> 59.8 mm, vias 0 -> 2
- net Net-(J1-Pin_4): track 0.00 -> 47.6 mm, vias 0 -> 2
- net Net-(J1-Pin_7): track 0.00 -> 45.4 mm, vias 0 -> 2
- net +5VA: track 0.00 -> 35.9 mm
- net Net-(J1-Pin_3): track 0.00 -> 34.5 mm, vias 0 -> 2
- net Net-(J1-Pin_6): track 0.00 -> 31.9 mm
- net /ADC_ParallelPort0: track 0.00 -> 29.5 mm
- net /AnalogComp_Out3: track 0.00 -> 28.5 mm, vias 0 -> 2
- net Net-(J1-Pin_5): track 0.00 -> 27.7 mm
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- added copper zone on B.Cu, net GND
- added copper zone on F.Cu, net GND
Other:
- board outline added: 90 x 90 mm
- board text added: "ESTA PLACA NO ESTA LISTA, REVISAR Y HACER UNA NUEVA VERSION"
