File: Placas/Placa Definitiva/v0.1/v0.1.kicad_sch (KiCad schematic)
At the start: 47 parts, among them IC1 SN74LVTH245ADWR, IC2 ADA4891-1ARJZ-RL, J1 Conn_01x09_Pin, Q1 BC807, Q2 BC807, Q3 BC807, Q4 BC807, Q5 BC807, Q6 BC807, Q7 BC807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

Commit message: skere
Parts:
- removed C10, C9: 100nF, symbol Device:C
- added C15: 10nF, Capacitor_SMD:C_0805_2012Metric_Pad1.18x1.45mm_HandSolder, symbol Device:C
- added J2: Screw_Terminal_01x02, TerminalBlock:TerminalBlock_bornier-2_P5.08mm, symbol Connector:Screw_Terminal_01x02
- added R5: 150k, Resistor_SMD:R_1206_3216Metric_Pad1.30x1.75mm_HandSolder, symbol Device:R
- C1, C12, C13, C3, C7: footprint (none) -> Capacitor_Tantalum_SMD:CP_EIA-3528-15_AVX-H_Pad1.50x2.35mm_HandSolder
- C11, C14, C2, C4, C6, C8: footprint (none) -> Capacitor_SMD:C_0805_2012Metric_Pad1.18x1.45mm_HandSolder
- C5: footprint (none) -> Capacitor_SMD:CP_Elec_6.3x7.7
- F1: footprint (none) -> Fuse:Fuse_1206_3216Metric_Pad1.42x1.75mm_HandSolder
- J1: footprint (none) -> Connector_PinHeader_2.54mm:PinHeader_1x09_P2.54mm_Vertical
- L1, L2: value 200uH -> 330uH; footprint (none) -> Inductor_SMD:L_Sunlord_SWRB1205S
- R1, R2: footprint Resistor_THT:R_Axial_DIN0411_L9.9mm_D3.6mm_P12.70mm_Horizontal -> Resistor_SMD:R_1206_3216Metric_Pad1.30x1.75mm_HandSolder
- R3, R4: value 100k -> 150k; footprint (none) -> Resistor_SMD:R_1206_3216Metric_Pad1.30x1.75mm_HandSolder
- U4: footprint (none) -> Package_SO:SOIC-8_3.9x4.9mm_P1.27mm
Connections:
- net +3.3V: now also R5.1
- net GND: now also C15.2, J2.1 (Pin_1)
- net ResetButton: now reaches U3.30 (~{RUN})
- net ResetButton: now also C15.1, J2.2 (Pin_2), R5.2
- no-connect marks 29 -> 28
Other:
- moved on the sheet: F1, U3
